Commit message: merge description and gazebo. add namespace

File: urdf/lidar_gazebo.xacro (robot description, xacro)
@@ -2,5 +2,5 @@
 <robot xmlns:xacro="http://www.ros.org/wiki/xacro" name="lidar">
         <!-- Create laser reference frame -->
- <gazebo reference="lidar_Link">
+ <gazebo reference="${tf_prefix}laser">
             <sensor type="ray" name="rplidar">
                 <pose>0 0 0 0 0 0</pose>
@@ -28,6 +28,7 @@
                 </ray>
                 <plugin name="gazebo_rplidar" filename="libgazebo_ros_laser.so">
-                    <topicName>/scan</topicName>
-                    <frameName>lidar_Link</frameName>
+                    <robotNamespace>/</robotNamespace>
+                    <topicName>${tf_prefix}scan</topicName>
+                    <frameName>${tf_prefix}laser</frameName>
                 </plugin>
             </sensor>

File: urdf/tianbot_mini.urdf.xacro (robot description, xacro)
@@ -1,6 +1,6 @@
 <?xml version="1.0" encoding="utf-8"?>
 <robot xmlns:xacro="http://www.ros.org/wiki/xacro">
-  <link  name="base_link"/>
-  <link name="chassis">
+  <link name="${tf_prefix}base_link"/>
+  <link name="${tf_prefix}chassis">
     <visual>
       <origin
@@ -29,8 +29,8 @@
    <joint name="base_link_joint" type="fixed">
     <origin xyz="0 0 0" rpy="0 0 0" />
-    <parent link="base_link" />
-    <child link="chassis" />
-  </joint>
-<link name="chassis_inertia">
+    <parent link="${tf_prefix}base_link" />
+    <child link="${tf_prefix}chassis" />
+  </joint>
+<link name="${tf_prefix}chassis_inertia">
   <inertial>
       <origin
@@ -50,9 +50,9 @@
     <joint name="chassis_inertia_joint" type="fixed">
     <origin xyz="0 0 0" rpy="0 0 0" />
-    <parent link="chassis" />
-    <child link="chassis_inertia" />
+    <parent link="${tf_prefix}chassis" />
+    <child link="${tf_prefix}chassis_inertia" />
     </joint>
   <link
-    name="left_wheel_link">
+    name="${tf_prefix}left_wheel_link">
     <inertial>
       <origin
@@ -100,12 +100,12 @@
       rpy="0 0 0" />
     <parent
-      link="chassis" />
-    <child
-      link="left_wheel_link" />
+      link="${tf_prefix}chassis" />
+    <child
+      link="${tf_prefix}left_wheel_link" />
     <axis
       xyz="0 1 0" />
   </joint>
   <link
-    name="right_wheel_link">
+    name="${tf_prefix}right_wheel_link">
     <inertial>
       <origin
@@ -153,12 +153,12 @@
       rpy="0 0 0" />
     <parent
-      link="chassis" />
-    <child
-      link="right_wheel_link" />
+      link="${tf_prefix}chassis" />
+    <child
+      link="${tf_prefix}right_wheel_link" />
     <axis
       xyz="0 1 0" />
   </joint>
   <link
-    name="caster_wheel_link">
+    name="${tf_prefix}caster_wheel_link">
     <inertial>
       <origin
@@ -206,12 +206,12 @@
       rpy="0 0 0" />
     <parent
-      link="chassis" />
-    <child
-      link="caster_wheel_link" />
+      link="${tf_prefix}chassis" />
+    <child
+      link="${tf_prefix}caster_wheel_link" />
     <axis
       xyz="0 0 -1" />
   </joint>
   <link
-    name="casterball_link">
+    name="${tf_prefix}casterball_link">
     <inertial>
       <origin
@@ -259,12 +259,12 @@
       rpy="0 0 0" />
     <parent
-      link="caster_wheel_link" />
-    <child
-      link="casterball_link" />
+      link="${tf_prefix}caster_wheel_link" />
+    <child
+      link="${tf_prefix}casterball_link" />
     <axis
       xyz="0.73589 -0.6771 0" />
   </joint>
   <link
-    name="lidar_Link">
+    name="${tf_prefix}laser">
     <inertial>
       <origin
@@ -312,21 +312,29 @@
       rpy="0 0 0" />
     <parent
-      link="base_link" />
-    <child
-      link="lidar_Link" />
+      link="${tf_prefix}base_link" />
+    <child
+      link="${tf_prefix}laser" />
     <axis
       xyz="0 0 0" />
   </joint>
-<gazebo reference="chassis">
+<gazebo reference="${tf_prefix}chassis">
      <material>Gazebo/Red </material>
+     <maxVel>0.0</maxVel>
+     <minDepth>0.001</minDepth>
     </gazebo>
- <gazebo reference="right_wheel_link">
+ <gazebo reference="${tf_prefix}right_wheel_link">
      <material>Gazebo/Black </material>
+     <maxVel>0.0</maxVel>
+     <minDepth>0.001</minDepth>
     </gazebo>
- <gazebo reference="left_wheel_link">
+ <gazebo reference="${tf_prefix}left_wheel_link">
      <material>Gazebo/Black </material>
+     <maxVel>0.0</maxVel>
+     <minDepth>0.001</minDepth>
     </gazebo>
- <gazebo reference="caster_wheel_link">
+ <gazebo reference="${tf_prefix}caster_wheel_link">
      <material>Gazebo/Blue </material>
+     <maxVel>0.0</maxVel>
+     <minDepth>0.001</minDepth>
     </gazebo>
  <!-- Transmission is important to link the joints and the controller -->
@@ -352,5 +360,5 @@
                 <publishTf>1</publishTf>
                 <publishOdomTF>true</publishOdomTF>
-                <publishWheelJointState>true</publishWheelJointState>
+                <publishWheelJointState>false</publishWheelJointState>
                 <alwaysOn>true</alwaysOn>
                 <updateRate>50.0</updateRate>
@@ -363,9 +371,9 @@
                 <wheelTorque>30</wheelTorque>
                 <wheelAcceleration>1.8</wheelAcceleration>
-                <commandTopic>tianbot_mini/cmd_vel</commandTopic>
-                <odometryFrame>tianbot_mini/odom</odometryFrame>
-                <odometryTopic>tianbot_mini/odom</odometryTopic>
+                <commandTopic>${tf_prefix}cmd_vel</commandTopic>
+                <odometryFrame>${tf_prefix}odom</odometryFrame>
+                <odometryTopic>${tf_prefix}odom</odometryTopic>
                 <odometrySource>world</odometrySource>
-                <robotBaseFrame>tianbot_mini/base_link</robotBaseFrame>
+                <robotBaseFrame>${tf_prefix}base_link</robotBaseFrame>
             </plugin>
         </gazebo>

File: urdf/tianbot_mini_run.urdf.xacro (robot description, xacro)
@@ -1,4 +1,11 @@
 <?xml version="1.0"?>
 <robot name="tianbot_mini" xmlns:xacro="http://www.ros.org/wiki/xacro">
+    <xacro:property name="prefix" value="$(arg prefix)" />
+    <xacro:if value="${prefix == '/' or prefix == '' or prefix == ' '}">
+    <xacro:property name="tf_prefix" value="" />
+    </xacro:if>
+    <xacro:unless value="${prefix == '/' or prefix == '' or prefix == ' '}">
+    <xacro:property name="tf_prefix" value="${prefix}/" />
+    </xacro:unless>
     <xacro:include filename="$(find tianbot_mini)/urdf/tianbot_mini.urdf.xacro" />
     <xacro:include filename="$(find tianbot_mini)/urdf/lidar_gazebo.xacro" />
